File: PCB/solenoid.kicad_pcb (KiCad board)
At the start: 2 copper layers, 15.8 x 25.7 mm, 7 parts, among them J1 esp32

Commit message: Add files via upload
Parts:
- moved r1 7.64 mm to (108.0, 116.0)
- moved r2 7.23 mm to (108.8, 105.0)
- moved J1 6.39 mm to (107.5, 135.5)
- moved 1N4007 5.46 mm to (108.0, 126.8)
- moved solenoid1 0.71 mm to (103.0, 113.0)
Routing:
- net Net-(J1-Pin_2): track 7.81 -> 31.3 mm, vias 1 -> 0
- net Net-(1N4007-K): track 29.6 -> 23.8 mm, vias 0 -> 1
- net Net-(IRLZ44N1-G): track 22.6 -> 27.7 mm
- net VCC: track 33.4 -> 33.0 mm, vias 2 -> 1
Other:
- board size 15.8 x 25.7 mm -> 11.8 x 35.2 mm
- board text added: "Made by z0hra1n"
- board text removed: "esp32"
